Commit message: Make the robot URDF a single tree so Foxglove renders it
Current Foxglove rejects robot.urdf: "URDF contains multiple frames
without parent joint ... but only one root frame is allowed". The four
links had no joints, and their colours used SDF tags (<ambient>,
<diffuse>) that URDF doesn't read.

robot/chassis is now the root, with continuous joints to the wheels and
a fixed joint to the caster at the poses from robot_env.sdf, and URDF
<material>/<color> colours (blue chassis, red wheels, green caster).
The file is only used for visualisation; the simulator loads
robot_env.sdf. The Foxglove layout now loads both URDFs from this
repository.

Co-Authored-By: Claude Opus 5.5 <noreply@anthropic.com>

File: src/gazebo/launch/robot.urdf (robot description, URDF)
Before this commit: robot robot, 4 links, 0 joints
Joints:
- added joint caster_joint: type fixed, parent robot/chassis, child robot/caster, origin xyz=0.8 0 -0.2
- added joint left_wheel_joint: type continuous, parent robot/chassis, child robot/left_wheel, origin xyz=-0.5 0.6 0 rpy=-1.5707 0 0, axis 0 0 1
- added joint right_wheel_joint: type continuous, parent robot/chassis, child robot/right_wheel, origin xyz=-0.5 -0.6 0 rpy=-1.5707 0 0, axis 0 0 1
